Commit message: Ultrasonic Added and RViz launch strengthened

File: gym-gazebo/gym_gazebo/envs/installation/active_ws/src/lsd/urdf/lsd.urdf (robot description, URDF)
Before this commit: robot lsd, 23 links, 22 joints
Links:
- added link ultrasonic, mass 1e-5; collision box size=0.03 0.03 0.03; visual box size=0.03 0.03 0.03
Joints:
- added joint ultrasonic_joint: type fixed, parent CH, child ultrasonic, origin xyz=0 0 -0.1 rpy=0 1.5707 0

Commit message: .

File: gym-gazebo/gym_gazebo/envs/installation/active_ws/src/lsd/urdf/lsd.urdf (robot description, URDF)
Before this commit: robot lsd, 24 links, 23 joints
Links:
- removed link color
- removed link depth
- removed link holder
- removed link ired1
- removed link ired2
- removed link lidar_box
- removed link rs200_camera
- removed link ultrasonic
Joints:
- removed joint color_joint
- removed joint depth_joint
- removed joint holder_joint
- removed joint ired1_joint
- removed joint ired2_joint
- removed joint lidar_box_joint
- removed joint realsense_joint
- removed joint ultrasonic_joint
